File: ThumbsUp.kicad_pcb (KiCad board)
At the start: 2 copper layers, 247.3 x 280.9 mm, 165 parts, among them IC1 RP2040, IC2 W25Q128JVSIM, IC3 RP2040, IC4 W25Q128JVSIM, J1 Conn_01x04_Male, J10 Raiser_Male, J11 Raiser_Female, J12 Raiser_Male, J13 Raiser_Female, J14 Raiser_Male, J15 Raiser_Female, J16 Raiser_Male, J17 Raiser_Female, J18 Raiser_Male, J19 Raiser_Female, J2 Conn_01x04_Male, J20 Conn_01x04_Female, J21 Conn_01x04_Female, J22 Conn_01x04_Female, J23 Conn_01x04_Female, J24 Conn_01x04_Male, J25 Conn_01x04_Male, J26 Conn_01x04_Male, J27 Conn_01x04_Male, J28 Conn_01x04_Female, J29 Conn_01x04_Female, J3 Conn_01x04_Female, J30 Conn_01x04_Female, J31 Conn_01x04_Female, J32 USB_C_Receptacle_USB2.0, J33 Raiser_Male, J34 Raiser_Female, J35 Raiser_Male, J36 STX-3501-3N, J37 USB_C_Receptacle_USB2.0, J38 Raiser_Female, J39 Raiser_Male, J4 Conn_01x04_Male, J40 Raiser_Female, J41 Raiser_Male, J42 Raiser_Female, J43 Raiser_Male, J44 Raiser_Female, J45 Raiser_Male, J46 STX-3501-3N, J47 Raiser_Female, J48 Raiser_Male, J5 Conn_01x04_Female, J6 Conn_01x04_Male, J7 Conn_01x04_Male, J8 Conn_01x04_Male, J9 Raiser_Female, U1 NCP1117-3.3_SOT223, U2 NCP1117-3.3_SOT223, Y1 ABLS-12.000MHZ-B4-T, Y2 ABLS-12.000MHZ-B4-T

Commit message: Enlarged the PCBs, rearranged the raisers.
Parts:
- moved J32 21.3 mm to (110.9, 372.7)
- moved J37 21.3 mm to (173.5, 372.6)
- moved J38 20.6 mm to (126.4, 507.2)
- moved J39 20.6 mm to (128.9, 379.7)
- moved J41 20.6 mm to (155.5, 379.4)
- moved J40 20.6 mm to (153.0, 506.9)
- moved J44 18.6 mm to (126.4, 557.3)
- moved J43 18.6 mm to (155.4, 429.7)
- moved J45 18.6 mm to (128.9, 429.8)
- moved J42 18.5 mm to (152.9, 557.2)
- moved J23 1.55 mm to (103.5, 556.5)
- moved J30 1.55 mm to (183.9, 537.3)
- moved J2 1.55 mm to (106.1, 390.8)
- moved J25 1.55 mm to (178.2, 390.9)
- moved J26 1.55 mm to (186.4, 409.8)
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Routing:
- net Net-(J22-Pad1): track 244.2 -> 506.2 mm
- net Net-(J44-Pad1): track 134.7 -> 0.00 mm
- net Net-(J44-Pad2): track 104.7 -> 0.00 mm
- net Net-(J42-Pad3): track 82.7 -> 0.00 mm
- net Net-(J30-Pad1): track 0.00 -> 82.7 mm
- net Net-(J21-Pad4): track 22.7 -> 0.00 mm
Other:
- board size 247.3 x 280.9 mm -> 250.9 x 280.9 mm

Commit message: Roughed in the lower plates
Parts:
- moved J46 22.3 mm to (157.8, 386.1)
- moved J36 22.0 mm to (125.9, 391.2)
- moved F1 2.20 mm to (112.2, 405.4), turned to 90 degrees
- moved J32 0.43 mm to (111.0, 373.2)
- moved J37 0.35 mm to (173.5, 373.0)
- turned MX15 to 180 degrees
- turned MX16 to 180 degrees
- turned MX17 to 180 degrees
- turned MX19 to 0 degrees
- turned MX23 to 0 degrees
- turned MX3 to 180 degrees
Connections:
- J2 pad 1: K_GRAVE -> K_3
- J2 pad 2: K_1 -> K_2
- J2 pad 3: K_2 -> K_1
- J2 pad 4: K_3 -> K_GRAVE
- J25 pad 1: K_8 -> K_DEL
- J25 pad 2: K_9 -> K_0
- J25 pad 3: K_0 -> K_9
- J25 pad 4: K_DEL -> K_8
- MX45 pad 2: Net-(J21-Pad1) -> Net-(J21-Pad4)
- MX46 pad 2: Net-(J21-Pad2) -> Net-(J21-Pad3)
- MX47 pad 2: Net-(J21-Pad3) -> Net-(J21-Pad2)
- MX48 pad 2: Net-(J21-Pad4) -> Net-(J21-Pad1)
- MX53 pad 2: Net-(J29-Pad4) -> Net-(J29-Pad1)
- MX54 pad 2: Net-(J29-Pad3) -> Net-(J29-Pad2)
- MX55 pad 2: Net-(J29-Pad2) -> Net-(J29-Pad3)
- MX56 pad 2: Net-(J29-Pad1) -> Net-(J29-Pad4)
Routing:
- net L-BASE: track 827.5 -> 309.5 mm, vias 30 -> 28
- net Net-(J30-Pad1): track 82.7 -> 566.4 mm
- net Net-(J29-Pad4): track 324.9 -> 100.1 mm
- net Net-(J44-Pad1): track 0.00 -> 122.2 mm
- net Net-(J44-Pad2): track 0.00 -> 95.6 mm
- net Net-(J21-Pad4): track 0.00 -> 85.9 mm
- net R-TIP: track 90.3 -> 7.18 mm, vias 3 -> 1
- net Net-(J29-Pad3): track 0.00 -> 81.9 mm
- net Net-(J42-Pad3): track 0.00 -> 79.7 mm
- net K_R: track 69.1 -> 0.00 mm
- net L-RING1: track 108.8 -> 44.6 mm
- net K_T: track 63.4 -> 0.00 mm
- net Net-(J29-Pad2): track 0.00 -> 63.3 mm
- net Net-(J21-Pad3): track 0.00 -> 61.2 mm
- net K_Y: track 60.6 -> 0.00 mm, vias 2 -> 0
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Other:
- outline, holes or cut-outs redrawn

Commit message: Routed R2
Parts:
- moved R10 28.6 mm to (179.0, 371.1), turned to 0 degrees
- moved R11 26.9 mm to (179.0, 372.2), turned to 180 degrees
- moved R5 20.7 mm to (166.2, 425.0), turned to 270 degrees
- moved U2 19.3 mm to (171.8, 424.9), turned to 0 degrees
- moved C8 17.9 mm to (170.4, 420.5)
- moved C18 15.5 mm to (166.2, 427.2), turned to 270 degrees
- moved F2 12.2 mm to (172.5, 388.3)
- moved J37 1.56 mm to (172.3, 372.1)
- moved C27 1.38 mm to (169.2, 452.5)
- moved Y2 1.19 mm to (186.3, 455.5)
- moved C32 0.96 mm to (175.7, 450.5)
- moved R15 0.59 mm to (170.3, 445.6)
- moved R14 0.58 mm to (171.3, 445.6)
- turned MX52 to 180 degrees
Connections:
- IC3 pad 11: K_U -> K_J
- IC3 pad 12: Net-(IC3-Pad12) -> K_6
- IC3 pad 13: Net-(IC3-Pad13) -> K_DEL
- IC3 pad 14: Net-(IC3-Pad14) -> K_0
- IC3 pad 27: Net-(IC3-Pad27) -> K_9
- IC3 pad 28: Net-(IC3-Pad28) -> K_8
- IC3 pad 35: Net-(IC3-Pad35) -> K_7
- IC3 pad 5: K_H -> K_Y
- IC3 pad 6: K_Y -> K_H
- IC3 pad 8: K_M -> K_U
- IC3 pad 9: K_J -> K_M
- J19 pad 1: Net-(J19-Pad1) -> L-BASE
- J19 pad 2: Net-(J19-Pad2) -> L-BASE
- J19 pad 3: Net-(J19-Pad3) -> L-BASE
- J24 pad 1: Net-(J24-Pad1) -> L-BASE
- J24 pad 2: Net-(J24-Pad2) -> L-BASE
- J24 pad 3: Net-(J24-Pad3) -> L-BASE
- J24 pad 4: Net-(J24-Pad4) -> L-BASE
- J34 pad 1: Net-(J34-Pad1) -> L-BASE
- J34 pad 2: Net-(J34-Pad2) -> L-BASE
- J34 pad 3: Net-(J34-Pad3) -> L-BASE
- J34 pad 4: Net-(J34-Pad4) -> L-BASE
Routing:
- net K_7: track 0.00 -> 133.8 mm, vias 0 -> 3
- net K_8: track 0.00 -> 107.8 mm, vias 0 -> 1
- net L-BASE: track 309.5 -> 417.1 mm
- net K_9: track 0.00 -> 105.2 mm, vias 0 -> 1
- net R-TIP: track 7.18 -> 107.1 mm, vias 1 -> 2
- net K_Y: track 0.00 -> 92.6 mm
- net K_6: track 0.00 -> 88.4 mm, vias 0 -> 2
- net RD-: track 0.00 -> 73.9 mm, vias 0 -> 2
- net K_BSPC: track 0.00 -> 73.7 mm, vias 0 -> 2
- net RD+: track 0.30 -> 73.4 mm, vias 0 -> 2
- net K_0: track 0.00 -> 72.5 mm, vias 0 -> 1
- net K_DEL: track 0.00 -> 70.7 mm, vias 0 -> 1
- net K_U: track 0.00 -> 65.7 mm, vias 0 -> 2
- net K_MNU: track 0.00 -> 59.9 mm
- net Net-(J6-Pad4): track 0.00 -> 55.9 mm
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- added copper zone on B.Cu, net L-BASE

Commit message: Routing L2
Parts:
- moved R2 37.4 mm to (141.3, 426.1)
- moved R1 37.4 mm to (140.2, 426.1)
- moved U1 22.0 mm to (116.1, 426.5), turned to 0 degrees
- moved R9 21.8 mm to (118.6, 372.5)
- moved R8 21.7 mm to (118.6, 371.5)
- moved C9 19.6 mm to (114.1, 422.2), turned to 0 degrees
- moved C11 19.5 mm to (110.9, 427.4), turned to 270 degrees
- moved J32 1.42 mm to (112.0, 372.2)
- turned MX15 to 0 degrees
- turned MX16 to 0 degrees
Connections:
- IC1 pad 5: K_LCTL -> K_C
- IC1 pad 6: K_Z -> K_X
- IC1 pad 7: K_X -> K_Z
- IC1 pad 8: K_C -> K_LCTL
- J1 pad 1: Net-(J1-Pad1) -> K_WIN
Routing:
- net K_WIN: track 0.00 -> 65.5 mm
- net K_LCTL: track 0.00 -> 46.4 mm, vias 0 -> 1
- net K_LALT: track 0.00 -> 46.2 mm
- net K_Z: track 0.00 -> 43.5 mm, vias 0 -> 1
- net K_X: track 0.00 -> 41.6 mm, vias 0 -> 1
- net K_C: track 0.10 -> 40.6 mm, vias 0 -> 1
- net L-RING1: track 90.8 -> 54.5 mm, vias 2 -> 1
- net K_V: track 0.10 -> 33.1 mm
- net L-BASE: track 417.1 -> 397.0 mm, vias 28 -> 27
- net +3V3: track 237.5 -> 227.6 mm
- net +1V1: track 56.0 -> 57.7 mm
- net Net-(IC1-Pad46): track 20.9 -> 20.2 mm

Commit message: Routing completed
Parts:
- added G***: LOGO, Silkscreens:Crowfeet75, F.Cu at (140.6, 557.8)
- added G***: LOGO, Silkscreens:Crowfeet75, B.Cu at (140.7, 557.9)
- added G***: LOGO, Silkscreens:Crowfeet75, B.Cu at (143.2, 398.6)
- moved R2 39.0 mm to (109.4, 448.6)
- moved R1 39.0 mm to (108.4, 448.6)
- moved F1 24.4 mm to (112.2, 380.9)
- moved R4 2.26 mm to (116.9, 469.4)
- moved C4 1.86 mm to (120.0, 458.8)
- moved C5 1.84 mm to (120.0, 459.8)
- moved R17 0.64 mm to (119.0, 467.4)
- moved C2 0.60 mm to (114.3, 467.7)
- moved C9 0.56 mm to (113.5, 422.1)
- moved Y1 0.49 mm to (124.3, 462.2)
Connections:
- IC1 pad 11: K_F -> K_R
- IC1 pad 27: Net-(IC1-Pad27) -> K_4
- IC1 pad 28: Net-(IC1-Pad28) -> K_5
- IC1 pad 30: Net-(IC1-Pad30) -> K_GRAVE
- IC1 pad 31: Net-(IC1-Pad31) -> K_1
- IC1 pad 34: Net-(IC1-Pad34) -> K_2
- IC1 pad 35: Net-(IC1-Pad35) -> K_3
- IC1 pad 9: K_R -> K_F
- J39 pad 1: Net-(J39-Pad1) -> K_5
Routing:
- net K_4: track 0.00 -> 122.9 mm, vias 0 -> 1
- net K_5: track 0.00 -> 122.0 mm, vias 0 -> 1
- net K_3: track 0.00 -> 102.5 mm, vias 0 -> 1
- net K_2: track 0.00 -> 101.6 mm, vias 0 -> 1
- net K_1: track 0.00 -> 99.3 mm, vias 0 -> 1
- net K_GRAVE: track 0.00 -> 99.3 mm, vias 0 -> 1
- net L-TIP: track 9.52 -> 101.2 mm
- net K_T: track 0.00 -> 86.1 mm, vias 0 -> 1
- net D-: track 0.00 -> 77.5 mm, vias 0 -> 2
- net D+: track 0.13 -> 77.6 mm, vias 0 -> 2
- net K_R: track 0.00 -> 69.8 mm, vias 0 -> 2
- net K_F: track 0.00 -> 56.2 mm, vias 0 -> 1
- net L-RING1: track 54.5 -> 106.4 mm, vias 1 -> 0
- net K_G: track 0.00 -> 51.3 mm, vias 0 -> 1
- net K_E: track 0.00 -> 46.1 mm, vias 0 -> 1
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
Commit message: Added a raiser near USB connectors
Parts:
- removed the G*** at (140.6, 557.8)
- removed the G*** at (140.7, 557.9)
- removed the G*** at (143.2, 398.6)
- added G***: LOGO, Silkscreens:Crowfeet75, F.Cu at (140.0, 556.3)
- added G***: LOGO, Silkscreens:Crowfeet75, B.Cu at (140.8, 560.0)
- added G***: LOGO, Silkscreens:Crowfeet75, F.Cu at (141.1, 398.2)
- added J49: Raiser_Female, Connector_PinSocket_2.54mm:PinSocket_1x04_P2.54mm_Vertical, F.Cu at (102.6, 498.3)
- added J50: Raiser_Male, Connector_PinHeader_2.54mm:PinHeader_1x04_P2.54mm_Vertical, B.Cu at (105.1, 370.8)
- added J51: Raiser_Female, Connector_PinSocket_2.54mm:PinSocket_1x04_P2.54mm_Vertical, F.Cu at (176.7, 498.4)
- added J52: Raiser_Male, Connector_PinHeader_2.54mm:PinHeader_1x04_P2.54mm_Vertical, B.Cu at (179.2, 370.9)
- moved R10 1.74 mm to (179.5, 372.7)
- moved R11 1.63 mm to (179.5, 373.7)
Routing:
- net Net-(J21-Pad4): track 85.9 -> 88.6 mm
- net Net-(J21-Pad3): track 61.2 -> 62.6 mm
- net Net-(J37-PadB5): track 6.43 -> 7.64 mm
- net Net-(J21-Pad2): track 46.0 -> 47.0 mm
- net Net-(J37-PadA5): track 10.0 -> 10.6 mm
