File: ThumbsUp.sch (KiCad schematic (older format))
At the start: 165 parts, among them IC1 RP2040, IC2 W25Q128JVSIM, IC3 RP2040, IC4 W25Q128JVSIM, J1 Conn_01x04_Male, J10 Raiser_Male, J11 Raiser_Female, J12 Raiser_Male, J13 Raiser_Female, J14 Raiser_Male, J15 Raiser_Female, J16 Raiser_Male, J17 Raiser_Female, J18 Raiser_Male, J19 Raiser_Female, J2 Conn_01x04_Male, J20 Conn_01x04_Female, J21 Conn_01x04_Female, J22 Conn_01x04_Female, J23 Conn_01x04_Female, J24 Conn_01x04_Male, J25 Conn_01x04_Male, J26 Conn_01x04_Male, J27 Conn_01x04_Male, J28 Conn_01x04_Female, J29 Conn_01x04_Female, J3 Conn_01x04_Female, J30 Conn_01x04_Female, J31 Conn_01x04_Female, J32 USB_C_Receptacle_USB2.0, J33 Raiser_Male, J34 Raiser_Female, J35 Raiser_Male, J36 STX-3501-3N, J37 USB_C_Receptacle_USB2.0, J38 Raiser_Female, J39 Raiser_Male, J4 Conn_01x04_Male, J40 Raiser_Female, J41 Raiser_Male, J42 Raiser_Female, J43 Raiser_Male, J44 Raiser_Female, J45 Raiser_Male, J46 STX-3501-3N, J47 Raiser_Female, J48 Raiser_Male, J5 Conn_01x04_Female, J6 Conn_01x04_Male, J7 Conn_01x04_Male, J8 Conn_01x04_Male, J9 Raiser_Female, U1 NCP1117-3.3_SOT223, U2 NCP1117-3.3_SOT223, Y1 ABLS-12.000MHZ-B4-T, Y2 ABLS-12.000MHZ-B4-T

Commit message: Routing completed
Connections:
- net K_1: now also IC1.31 (GPIO20)
- net K_2: now also IC1.34 (GPIO22)
- net K_3: now also IC1.35 (GPIO23)
- net K_4: now also IC1.27 (GPIO16)
- net K_5: now also IC1.28 (GPIO17), J39.1 (Pin_1)
- net K_F: now also IC1.9 (GPIO7); no longer IC1.11 (GPIO8)
- net K_GRAVE: now also IC1.30 (GPIO19)
- net K_R: now also IC1.11 (GPIO8); no longer IC1.9 (GPIO7)
- no-connect marks 77 -> 78
Other:
- moved on the sheet: J36, R4, RUN1
Changed lines of the file:
@@
 L power:GND #PWR0117
 U 1 1 63E16CE5
-P 3850 10150
-F 0 "#PWR0117" H 3850 9900 50  0001 C CNN
-F 1 "GND" H 3855 9977 50  0000 C CNN
-F 2 "" H 3850 10150 50  0001 C CNN
-F 3 "" H 3850 10150 50  0001 C CNN
-	1    3850 10150
+P 3850 10400
+F 0 "#PWR0117" H 3850 10150 50  0001 C CNN
+F 1 "GND" H 3855 10227 50  0000 C CNN
+F 2 "" H 3850 10400 50  0001 C CNN
+F 3 "" H 3850 10400 50  0001 C CNN
+	1    3850 10400
 	1    0    0    -1
 $EndComp
@@
 L TL1016AAF220QG:TL1016AAF220QG RUN1
 U 1 1 639D06EF
-P 4050 9350
-F 0 "RUN1" V 4450 9600 50  0000 L CNN
-F 1 "TL1016AAF220QG" V 4600 9600 50  0000 L CNN
-F 2 "TL1016AAF220QG:TL1016AAF220QG" H 4700 9450 50  0001 L CNN
-F 3 "https://eu.mouser.com/datasheet/2/140/E_Switch_05112022_TL1016_Datasheet-2943618.pdf" H 4700 9350 50  0001 L CNN
-F 4 "Tactile Switches Tactile Switch SPST OFF-(ON) 50mA 12VDC" H 4700 9250 50  0001 L CNN "Description"
-F 5 "1.35" H 4700 9150 50  0001 L CNN "Height"
-F 6 "E-Switch" H 4700 9050 50  0001 L CNN "Manufacturer_Name"
-F 7 "TL1016AAF220QG" H 4700 8950 50  0001 L CNN "Manufacturer_Part_Number"
-F 8 "612-TL1016AAF220QG" H 4700 8850 50  0001 L CNN "Mouser Part Number"
-F 9 "https://www.mouser.co.uk/ProductDetail/E-Switch/TL1016AAF220QG?qs=t7xnP681wgW5zrSpkWH91Q%3D%3D" H 4700 8750 50  0001 L CNN "Mouser Price/Stock"
-F 10 "" H 4700 8650 50  0001 L CNN "Arrow Part Number"
-F 11 "" H 4700 8550 50  0001 L CNN "Arrow Price/Stock"
-F 12 "" H 4700 8450 50  0001 L CNN "Mouser Testing Part Number"
-F 13 "" H 4700 8350 50  0001 L CNN "Mouser Testing Price/Stock"
-	1    4050 9350
+P 4050 9600
+F 0 "RUN1" V 4450 9850 50  0000 L CNN
+F 1 "TL1016AAF220QG" V 4600 9850 50  0000 L CNN
+F 2 "TL1016AAF220QG:TL1016AAF220QG" H 4700 9700 50  0001 L CNN
+F 3 "https://eu.mouser.com/datasheet/2/140/E_Switch_05112022_TL1016_Datasheet-2943618.pdf" H 4700 9600 50  0001 L CNN
+F 4 "Tactile Switches Tactile Switch SPST OFF-(ON) 50mA 12VDC" H 4700 9500 50  0001 L CNN "Description"
+F 5 "1.35" H 4700 9400 50  0001 L CNN "Height"
+F 6 "E-Switch" H 4700 9300 50  0001 L CNN "Manufacturer_Name"
+F 7 "TL1016AAF220QG" H 4700 9200 50  0001 L CNN "Manufacturer_Part_Number"
+F 8 "612-TL1016AAF220QG" H 4700 9100 50  0001 L CNN "Mouser Part Number"
+F 9 "https://www.mouser.co.uk/ProductDetail/E-Switch/TL1016AAF220QG?qs=t7xnP681wgW5zrSpkWH91Q%3D%3D" H 4700 9000 50  0001 L CNN "Mouser Price/Stock"
+F 10 "" H 4700 8900 50  0001 L CNN "Arrow Part Number"
+F 11 "" H 4700 8800 50  0001 L CNN "Arrow Price/Stock"
+F 12 "" H 4700 8700 50  0001 L CNN "Mouser Testing Part Number"
+F 13 "" H 4700 8600 50  0001 L CNN "Mouser Testing Price/Stock"
+	1    4050 9600
 	0    1    1    0
 $EndComp
 Wire Wire Line
-	4050 9350 4150 9350
-Wire Wire Line
-	4200 9350 4200 10150
-Wire Wire Line
-	3750 10150 3850 10150
+	4050 9600 4150 9600
+Wire Wire Line
+	4200 9600 4200 10400
+Wire Wire Line
+	3750 10400 3850 10400
 $Comp
 L TL1016AAF220QG:TL1016AAF220QG BOOTSEL1
@@
 Connection ~ 2350 2000
 Wire Wire Line
-	3750 10150 3750 9350
-Wire Wire Line
-	3750 9350 3950 9350
+	3750 10400 3750 9600
+Wire Wire Line
+	3750 9600 3950 9600
 Wire Wire Line
 	4300 14400 4300 14150
@@
 NoConn ~ 20350 10400
 NoConn ~ 20450 10400
-NoConn ~ 20550 10400
 $Comp
 L Connector:Conn_01x04_Female J42
@@
 L power:GND #PWR0149
 U 1 1 641658E3
-P 5200 8100
-F 0 "#PWR0149" H 5200 7850 50  0001 C CNN
-F 1 "GND" H 5205 7927 50  0000 C CNN
-F 2 "" H 5200 8100 50  0001 C CNN
-F 3 "" H 5200 8100 50  0001 C CNN
-	1    5200 8100
-	1    0    0    -1
-$EndComp
-Wire Wire Line
-	5000 8100 5200 8100
-Wire Wire Line
-	5000 8900 5200 8900
-Text GLabel 4750 8100 3    50   Input ~ 0
+P 5500 8100
+F 0 "#PWR0149" H 5500 7850 50  0001 C CNN
+F 1 "GND" H 5505 7927 50  0000 C CNN
+F 2 "" H 5500 8100 50  0001 C CNN
+F 3 "" H 5500 8100 50  0001 C CNN
+	1    5500 8100
+	1    0    0    -1
+$EndComp
+Wire Wire Line
+	5300 8100 5500 8100
+Wire Wire Line
+	5300 8900 5500 8900
+Text GLabel 5050 8100 3    50   Input ~ 0
 L-TIP
-Text GLabel 5200 8100 2    50   Input ~ 0
+Text GLabel 5500 8100 2    50   Input ~ 0
 L-BASE
-Text GLabel 5200 8900 2    50   Input ~ 0
+Text GLabel 5500 8900 2    50   Input ~ 0
 L-RING1
 $Comp
@@
 L power:+5V #PWR0147
 U 1 1 63F119E5
-P 5000 8900
-F 0 "#PWR0147" H 5000 8750 50  0001 C CNN
-F 1 "+5V" H 5015 9073 50  0000 C CNN
-F 2 "" H 5000 8900 50  0001 C CNN
-F 3 "" H 5000 8900 50  0001 C CNN
-	1    5000 8900
+P 5300 8900
+F 0 "#PWR0147" H 5300 8750 50  0001 C CNN
+F 1 "+5V" H 5315 9073 50  0000 C CNN
+F 2 "" H 5300 8900 50  0001 C CNN
+F 3 "" H 5300 8900 50  0001 C CNN
+	1    5300 8900
 	-1   0    0    1
 $EndComp
-Connection ~ 5000 8900
+Connection ~ 5300 8900
 Wire Wire Line
 	4250 8000 5200 8000
@@
 L STX-3501-3N:STX-3501-3N J36
 U 1 1 63D573AD
-P 5000 8100
-F 0 "J36" V 5354 8228 50  0000 L CNN
-F 1 "STX-3501-3N" V 5445 8228 50  0000 L CNN
-F 2 "STX-3501-3N:STX35013N" H 5650 8200 50  0001 L CNN
-F 3 "https://datasheet.datasheetarchive.com/originals/distributors/Datasheets_SAMA/ae9d1df0991347f2f81145ba35ca04dc.pdf" H 5650 8100 50  0001 L CNN
-F 4 "Phone Connectors 3.5mm S LUGS STEREO 3P THRU HOLE" H 5650 8000 50  0001 L CNN "Description"
-F 5 "5" H 5650 7900 50  0001 L CNN "Height"
-F 6 "Kycon" H 5650 7800 50  0001 L CNN "Manufacturer_Name"
-F 7 "STX-3501-3N" H 5650 7700 50  0001 L CNN "Manufacturer_Part_Number"
-F 8 "806-STX-3501-3N" H 5650 7600 50  0001 L CNN "Mouser Part Number"
-F 9 "https://www.mouser.co.uk/ProductDetail/Kycon/STX-3501-3N?qs=BBNwCsfFaznpJt4o1Jp%2FTg%3D%3D" H 5650 7500 50  0001 L CNN "Mouser Price/Stock"
-F 10 "" H 5650 7400 50  0001 L CNN "Arrow Part Number"
-F 11 "" H 5650 7300 50  0001 L CNN "Arrow Price/Stock"
-F 12 "" H 5650 7200 50  0001 L CNN "Mouser Testing Part Number"
-F 13 "" H 5650 7100 50  0001 L CNN "Mouser Testing Price/Stock"
-	1    5000 8100
+P 5300 8100
+F 0 "J36" V 5654 8228 50  0000 L CNN
+F 1 "STX-3501-3N" V 5745 8228 50  0000 L CNN
+F 2 "STX-3501-3N:STX35013N" H 5950 8200 50  0001 L CNN
+F 3 "https://datasheet.datasheetarchive.com/originals/distributors/Datasheets_SAMA/ae9d1df0991347f2f81145ba35ca04dc.pdf" H 5950 8100 50  0001 L CNN
+F 4 "Phone Connectors 3.5mm S LUGS STEREO 3P THRU HOLE" H 5950 8000 50  0001 L CNN "Description"
+F 5 "5" H 5950 7900 50  0001 L CNN "Height"
+F 6 "Kycon" H 5950 7800 50  0001 L CNN "Manufacturer_Name"
+F 7 "STX-3501-3N" H 5950 7700 50  0001 L CNN "Manufacturer_Part_Number"
+F 8 "806-STX-3501-3N" H 5950 7600 50  0001 L CNN "Mouser Part Number"
+F 9 "https://www.mouser.co.uk/ProductDetail/Kycon/STX-3501-3N?qs=BBNwCsfFaznpJt4o1Jp%2FTg%3D%3D" H 5950 7500 50  0001 L CNN "Mouser Price/Stock"
+F 10 "" H 5950 7400 50  0001 L CNN "Arrow Part Number"
+F 11 "" H 5950 7300 50  0001 L CNN "Arrow Price/Stock"
+F 12 "" H 5950 7200 50  0001 L CNN "Mouser Testing Part Number"
+F 13 "" H 5950 7100 50  0001 L CNN "Mouser Testing Price/Stock"
+	1    5300 8100
 	0    1    1    0
 $EndComp
@@
 L Device:R R4
 U 1 1 63C3C97D
-P 4650 8250
-F 0 "R4" H 4720 8296 50  0000 L CNN
-F 1 "5.1K" H 4720 8205 50  0000 L CNN
-F 2 "Resistor_SMD:R_0402_1005Metric" V 4580 8250 50  0001 C CNN
-F 3 "~" H 4650 8250 50  0001 C CNN
-	1    4650 8250
-	-1   0    0    1
-$EndComp
-$Comp
-L power:+3.3V #PWR0150
-U 1 1 63C3E3CC
-P 4650 8400
-F 0 "#PWR0150" H 4650 8250 50  0001 C CNN
-F 1 "+3.3V" H 4665 8573 50  0000 C CNN
-F 2 "" H 4650 8400 50  0001 C CNN
-F 3 "" H 4650 8400 50  0001 C CNN
-	1    4650 8400
+P 4850 8250
+F 0 "R4" H 4920 8296 50  0000 L CNN
+F 1 "5.1K" H 4920 8205 50  0000 L CNN
+F 2 "Resistor_SMD:R_0402_1005Metric" V 4780 8250 50  0001 C CNN
+F 3 "~" H 4850 8250 50  0001 C CNN
+	1    4850 8250
 	-1   0    0    1
 $EndComp
@@
 	14050 10500 14050 9700
 Wire Wire Line
-	3650 9200 3650 9300
-Wire Wire Line
-	3650 9300 4150 9300
-Wire Wire Line
-	4150 9300 4150 9350
-Connection ~ 4150 9350
-Wire Wire Line
-	4150 9350 4200 9350
-Connection ~ 3850 10150
-Wire Wire Line
-	3850 10150 3950 10150
-Wire Wire Line
-	4050 10150 4200 10150
+	3650 9550 4150 9550
+Wire Wire Line
+	4150 9550 4150 9600
+Connection ~ 4150 9600
+Wire Wire Line
+	4150 9600 4200 9600
+Connection ~ 3850 10400
+Wire Wire Line
+	3850 10400 3950 10400
+Wire Wire Line
+	4050 10400 4200 10400
 Wire Wire Line
 	13950 9650 14400 9650
@@
 Text GLabel 2750 9200 3    50   Input ~ 0
 K_Q
-Wire Wire Line
-	4250 8100 4650 8100
-Connection ~ 4650 8100
-Wire Wire Line
-	4650 8100 4900 8100
 Text GLabel 2650 9200 3    50   Input ~ 0
 K_W
@@
 Text GLabel 2250 8200 0    50   Input ~ 0
 K_T
+Text GLabel 2250 7900 0    50   Input ~ 0
+K_F
 Text GLabel 2250 8100 0    50   Input ~ 0
-K_F
-Text GLabel 2250 7900 0    50   Input ~ 0
 K_R
 Text GLabel 2250 7400 0    50   Input ~ 0
@@
 Text GLabel 5600 15050 2    50   Input ~ 0
 K_WIN
+NoConn ~ 3450 9200
+NoConn ~ 3550 9200
+Text GLabel 4250 8200 2    50   Input ~ 0
+K_1
+Text GLabel 4250 7900 2    50   Input ~ 0
+K_2
+$Comp
+L power:+3.3V #PWR0150
+U 1 1 63C3E3CC
+P 4850 8400
+F 0 "#PWR0150" H 4850 8250 50  0001 C CNN
+F 1 "+3.3V" H 4865 8573 50  0000 C CNN
+F 2 "" H 4850 8400 50  0001 C CNN
+F 3 "" H 4850 8400 50  0001 C CNN
+	1    4850 8400
+	-1   0    0    1
+$EndComp
+Wire Wire Line
+	4250 8100 4850 8100
+Connection ~ 4850 8100
+Wire Wire Line
+	4850 8100 5200 8100
+Text GLabel 4250 7800 2    50   Input ~ 0
+K_3
+Text GLabel 4250 8300 2    50   Input ~ 0
+K_GRAVE
+Wire Wire Line
+	3650 9200 3650 9550
+Text GLabel 3850 9200 3    50   Input ~ 0
+K_5
+Text GLabel 3750 9200 3    50   Input ~ 0
+K_4
+Text GLabel 20550 10400 3    50   Input ~ 0
+K_5
 $EndSCHEMATC

Commit message: Added a raiser near USB connectors
Parts:
- added J49, J51: Raiser_Female, Connector_PinSocket_2.54mm:PinSocket_1x04_P2.54mm_Vertical, symbol Connector:Conn_01x04_Female
- added J50, J52: Raiser_Male, Connector_PinHeader_2.54mm:PinHeader_1x04_P2.54mm_Vertical, symbol Connector:Conn_01x04_Male
Connections:
- no-connect marks 78 -> 86
Other:
- moved on the sheet: J17, J18, J47, J48
Changed lines of the file:
@@
 L Connector:Conn_01x04_Female J17
 U 1 1 63ADD1E9
-P 18200 13550
-F 0 "J17" V 18046 13698 50  0000 L CNN
-F 1 "Raiser_Female" V 18137 13698 50  0000 L CNN
-F 2 "Connector_PinSocket_2.54mm:PinSocket_1x04_P2.54mm_Vertical" H 18200 13550 50  0001 C CNN
-F 3 "~" H 18200 13550 50  0001 C CNN
-	1    18200 13550
+P 18100 13450
+F 0 "J17" V 17946 13598 50  0000 L CNN
+F 1 "Raiser_Female" V 18037 13598 50  0000 L CNN
+F 2 "Connector_PinSocket_2.54mm:PinSocket_1x04_P2.54mm_Vertical" H 18100 13450 50  0001 C CNN
+F 3 "~" H 18100 13450 50  0001 C CNN
+	1    18100 13450
 	0    1    1    0
 $EndComp
@@
 L Connector:Conn_01x04_Male J18
 U 1 1 63ADD1EF
-P 18200 13700
-F 0 "J18" V 18262 13844 50  0000 L CNN
-F 1 "Raiser_Male" V 18353 13844 50  0000 L CNN
-F 2 "Connector_PinHeader_2.54mm:PinHeader_1x04_P2.54mm_Vertical" H 18200 13700 50  0001 C CNN
-F 3 "~" H 18200 13700 50  0001 C CNN
-	1    18200 13700
+P 18100 13600
+F 0 "J18" V 18162 13744 50  0000 L CNN
+F 1 "Raiser_Male" V 18253 13744 50  0000 L CNN
+F 2 "Connector_PinHeader_2.54mm:PinHeader_1x04_P2.54mm_Vertical" H 18100 13600 50  0001 C CNN
+F 3 "~" H 18100 13600 50  0001 C CNN
+	1    18100 13600
 	0    1    1    0
 $EndComp
-NoConn ~ 18000 13350
-NoConn ~ 18100 13350
-NoConn ~ 18200 13350
-NoConn ~ 18300 13350
-NoConn ~ 18000 13900
-NoConn ~ 18100 13900
-NoConn ~ 18200 13900
-NoConn ~ 18300 13900
+NoConn ~ 17900 13250
+NoConn ~ 18000 13250
+NoConn ~ 18100 13250
+NoConn ~ 18200 13250
+NoConn ~ 17900 13800
+NoConn ~ 18000 13800
+NoConn ~ 18100 13800
+NoConn ~ 18200 13800
 $Comp
 L power:GND #PWR0119
@@
 	-1   0    0    1
 $EndComp
-NoConn ~ 21400 9900
-NoConn ~ 21500 9900
-NoConn ~ 21600 9900
-NoConn ~ 21700 9900
-NoConn ~ 21400 10450
-NoConn ~ 21500 10450
-NoConn ~ 21600 10450
-NoConn ~ 21700 10450
 $Comp
 L Connector:Conn_01x04_Female J44
@@
 L Connector:Conn_01x04_Female J47
 U 1 1 63AC0C46
-P 18150 12650
-F 0 "J47" V 17996 12798 50  0000 L CNN
-F 1 "Raiser_Female" V 18087 12798 50  0000 L CNN
-F 2 "Connector_PinSocket_2.54mm:PinSocket_1x04_P2.54mm_Vertical" H 18150 12650 50  0001 C CNN
-F 3 "~" H 18150 12650 50  0001 C CNN
-	1    18150 12650
+P 18050 12550
+F 0 "J47" V 17896 12698 50  0000 L CNN
+F 1 "Raiser_Female" V 17987 12698 50  0000 L CNN
+F 2 "Connector_PinSocket_2.54mm:PinSocket_1x04_P2.54mm_Vertical" H 18050 12550 50  0001 C CNN
+F 3 "~" H 18050 12550 50  0001 C CNN
+	1    18050 12550
 	0    1    1    0
 $EndComp
@@
 L Connector:Conn_01x04_Male J48
 U 1 1 63AC0C4C
-P 18150 12800
-F 0 "J48" V 18212 12944 50  0000 L CNN
-F 1 "Raiser_Male" V 18303 12944 50  0000 L CNN
-F 2 "Connector_PinHeader_2.54mm:PinHeader_1x04_P2.54mm_Vertical" H 18150 12800 50  0001 C CNN
-F 3 "~" H 18150 12800 50  0001 C CNN
-	1    18150 12800
+P 18050 12700
+F 0 "J48" V 18112 12844 50  0000 L CNN
+F 1 "Raiser_Male" V 18203 12844 50  0000 L CNN
+F 2 "Connector_PinHeader_2.54mm:PinHeader_1x04_P2.54mm_Vertical" H 18050 12700 50  0001 C CNN
+F 3 "~" H 18050 12700 50  0001 C CNN
+	1    18050 12700
 	0    1    1    0
 $EndComp
-NoConn ~ 17950 12450
-NoConn ~ 18050 12450
-NoConn ~ 18150 12450
-NoConn ~ 18250 12450
-NoConn ~ 17950 13000
-NoConn ~ 18050 13000
-NoConn ~ 18150 13000
-NoConn ~ 18250 13000
+NoConn ~ 17850 12350
+NoConn ~ 17950 12350
+NoConn ~ 18050 12350
+NoConn ~ 18150 12350
+NoConn ~ 17850 12900
+NoConn ~ 17950 12900
+NoConn ~ 18050 12900
+NoConn ~ 18150 12900
 $Comp
 L Connector:Conn_01x04_Male J24
@@
 Text GLabel 20550 10400 3    50   Input ~ 0
 K_5
+$Comp
+L Connector:Conn_01x04_Female J51
+U 1 1 64043CBA
+P 18800 10900
+F 0 "J51" V 18646 11048 50  0000 L CNN
+F 1 "Raiser_Female" V 18737 11048 50  0000 L CNN
+F 2 "Connector_PinSocket_2.54mm:PinSocket_1x04_P2.54mm_Vertical" H 18800 10900 50  0001 C CNN
+F 3 "~" H 18800 10900 50  0001 C CNN
+	1    18800 10900
+	0    1    1    0
+$EndComp
+$Comp
+L Connector:Conn_01x04_Male J52
+U 1 1 64043CC0
+P 18800 11050
+F 0 "J52" V 18862 11194 50  0000 L CNN
+F 1 "Raiser_Male" V 18953 11194 50  0000 L CNN
+F 2 "Connector_PinHeader_2.54mm:PinHeader_1x04_P2.54mm_Vertical" H 18800 11050 50  0001 C CNN
+F 3 "~" H 18800 11050 50  0001 C CNN
+	1    18800 11050
+	0    1    1    0
+$EndComp
+NoConn ~ 18600 10700
+NoConn ~ 18700 10700
+NoConn ~ 18800 10700
+NoConn ~ 18900 10700
+NoConn ~ 18600 11250
+NoConn ~ 18700 11250
+NoConn ~ 18800 11250
+NoConn ~ 18900 11250
+$Comp
+L Connector:Conn_01x04_Female J49
+U 1 1 64043CCE
+P 18750 10000
+F 0 "J49" V 18596 10148 50  0000 L CNN
+F 1 "Raiser_Female" V 18687 10148 50  0000 L CNN
+F 2 "Connector_PinSocket_2.54mm:PinSocket_1x04_P2.54mm_Vertical" H 18750 10000 50  0001 C CNN
+F 3 "~" H 18750 10000 50  0001 C CNN
+	1    18750 10000
+	0    1    1    0
+$EndComp
+$Comp
+L Connector:Conn_01x04_Male J50
+U 1 1 64043CD4
+P 18750 10150
+F 0 "J50" V 18812 10294 50  0000 L CNN
+F 1 "Raiser_Male" V 18903 10294 50  0000 L CNN
+F 2 "Connector_PinHeader_2.54mm:PinHeader_1x04_P2.54mm_Vertical" H 18750 10150 50  0001 C CNN
+F 3 "~" H 18750 10150 50  0001 C CNN
+	1    18750 10150
+	0    1    1    0
+$EndComp
+NoConn ~ 18550 9800
+NoConn ~ 18650 9800
+NoConn ~ 18750 9800
+NoConn ~ 18850 9800
+NoConn ~ 18550 10350
+NoConn ~ 18650 10350
+NoConn ~ 18750 10350
+NoConn ~ 18850 10350
 $EndSCHEMATC
